Commit message: Add steering, ackermann plugin, and drive-in-a-circle launch
URDF additions:
- steered_wheel macro adds a small kingpin link + revolute steer joint
  for the front wheels (limit ~30 deg).
- Rear wheels still attach directly to base_link (driven).
- Gazebo <plugin> block embeds gz-sim-ackermann-steering-system, which
  reads gz.msgs.Twist on the 'cmd_vel' topic and computes per-wheel
  speeds + per-side steer angles using the wheelbase/track values.

ros_gz_bridge config (config/ros_gz_bridge.yaml) forwards ROS
/cmd_vel (geometry_msgs/Twist) to the Gazebo /cmd_vel topic.

Launch:
- spawn.launch.py now also starts the parameter_bridge.
- circle.launch.py includes spawn + a delayed (5 s, so Gazebo has time
  to come up) ros2 topic pub of Twist(linear=0.5, angular=0.5) at 10 Hz,
  giving a ~1 m radius circle.

Verified locally: workspace builds, xacro produces 6 joints, plugin
filename matches the installed libgz-sim-ackermann-steering-system.so.
Visual confirmation of actual driving needs X11 forwarding and is
deferred to user inspection.

File: ros/src/havoc_description/urdf/havoc.urdf.xacro (robot description, xacro)
@@ -11,4 +11,6 @@
   <xacro:property name="wheelbase" value="0.265"/>
   <xacro:property name="track"     value="0.21"/>
+  <!-- Max steering angle: ~30 deg, typical for a 1/10 RC. -->
+  <xacro:property name="steer_limit" value="0.524"/>
   <xacro:macro name="box_inertia" params="m x y z">
     <inertial>
@@ -27,15 +29,19 @@
     </inertial>
   </xacro:macro>
+  <xacro:macro name="wheel_visual_collision">
+    <visual>
+      <origin rpy="1.5708 0 0"/>
+      <geometry><cylinder radius="${wheel_radius}" length="${wheel_width}"/></geometry>
+      <material name="black"><color rgba="0.1 0.1 0.1 1"/></material>
+    </visual>
+    <collision>
+      <origin rpy="1.5708 0 0"/>
+      <geometry><cylinder radius="${wheel_radius}" length="${wheel_width}"/></geometry>
+    </collision>
+  </xacro:macro>
+  <!-- Rear (driven) wheel: continuous joint attached directly to base_link. -->
   <xacro:macro name="wheel" params="name x y">
     <link name="${name}_link">
-      <visual>
-        <origin rpy="1.5708 0 0"/>
-        <geometry><cylinder radius="${wheel_radius}" length="${wheel_width}"/></geometry>
-        <material name="black"><color rgba="0.1 0.1 0.1 1"/></material>
-      </visual>
-      <collision>
-        <origin rpy="1.5708 0 0"/>
-        <geometry><cylinder radius="${wheel_radius}" length="${wheel_width}"/></geometry>
-      </collision>
+      <xacro:wheel_visual_collision/>
       <xacro:cyl_inertia m="${wheel_mass}" r="${wheel_radius}" l="${wheel_width}"/>
     </link>
@@ -44,4 +50,30 @@
       <child  link="${name}_link"/>
       <origin xyz="${x} ${y} ${wheel_radius}"/>
+      <axis xyz="0 1 0"/>
+    </joint>
+  </xacro:macro>
+  <!-- Front (steered) wheel: kingpin link + revolute steer joint + continuous wheel joint. -->
+  <xacro:macro name="steered_wheel" params="name x y">
+    <link name="${name}_steer_link">
+      <inertial>
+        <mass value="0.05"/>
+        <inertia ixx="1e-5" ixy="0" ixz="0" iyy="1e-5" iyz="0" izz="1e-5"/>
+      </inertial>
+    </link>
+    <joint name="${name}_steer_joint" type="revolute">
+      <parent link="base_link"/>
+      <child  link="${name}_steer_link"/>
+      <origin xyz="${x} ${y} ${wheel_radius}"/>
+      <axis xyz="0 0 1"/>
+      <limit lower="${-steer_limit}" upper="${steer_limit}" effort="2.0" velocity="3.0"/>
+    </joint>
+    <link name="${name}_link">
+      <xacro:wheel_visual_collision/>
+      <xacro:cyl_inertia m="${wheel_mass}" r="${wheel_radius}" l="${wheel_width}"/>
+    </link>
+    <joint name="${name}_joint" type="continuous">
+      <parent link="${name}_steer_link"/>
+      <child  link="${name}_link"/>
+      <origin xyz="0 0 0"/>
       <axis xyz="0 1 0"/>
     </joint>
@@ -59,7 +91,24 @@
     <xacro:box_inertia m="${body_mass}" x="${body_length}" y="${body_width}" z="${body_height}"/>
   </link>
-  <xacro:wheel name="front_left"  x="${ wheelbase/2.0}" y="${ track/2.0}"/>
-  <xacro:wheel name="front_right" x="${ wheelbase/2.0}" y="${-track/2.0}"/>
-  <xacro:wheel name="rear_left"   x="${-wheelbase/2.0}" y="${ track/2.0}"/>
-  <xacro:wheel name="rear_right"  x="${-wheelbase/2.0}" y="${-track/2.0}"/>
+  <xacro:steered_wheel name="front_left"  x="${ wheelbase/2.0}" y="${ track/2.0}"/>
+  <xacro:steered_wheel name="front_right" x="${ wheelbase/2.0}" y="${-track/2.0}"/>
+  <xacro:wheel         name="rear_left"   x="${-wheelbase/2.0}" y="${ track/2.0}"/>
+  <xacro:wheel         name="rear_right"  x="${-wheelbase/2.0}" y="${-track/2.0}"/>
+  <!-- Gazebo ackermann_steering plugin: drives rear wheels, steers front wheels,
+       listens on the gz topic 'cmd_vel' for Twist messages. -->
+  <gazebo>
+    <plugin filename="gz-sim-ackermann-steering-system"
+            name="gz::sim::systems::AckermannSteering">
+      <left_joint>rear_left_joint</left_joint>
+      <right_joint>rear_right_joint</right_joint>
+      <left_steering_joint>front_left_steer_joint</left_steering_joint>
+      <right_steering_joint>front_right_steer_joint</right_steering_joint>
+      <kingpin_width>${track}</kingpin_width>
+      <steering_limit>${steer_limit}</steering_limit>
+      <wheel_base>${wheelbase}</wheel_base>
+      <wheel_separation>${track}</wheel_separation>
+      <wheel_radius>${wheel_radius}</wheel_radius>
+      <topic>cmd_vel</topic>
+    </plugin>
+  </gazebo>
 </robot>

Commit message: Phase 0: add depth camera + IMU to URDF, bridge sensor topics
First step of the Autonomy Plan. Wires the sensors SLAM and perception
will consume in later phases (RTAB-Map, Nav2, target detection).

- urdf/havoc.urdf.xacro: new camera_link + camera_optical_link pair
  (robot frame -> optical frame, per REP-103) mounted at the front of
  the chassis where the RealSense D435i will live, tilted ~10 deg down.
  Gazebo rgbd_camera sensor block publishes RGB + depth + cloud +
  camera_info on /camera/* at 30 Hz, 640x480, 69 deg FOV to match the
  real D435i. Also a new imu_link at chassis center with a 200 Hz IMU
  sensor.

- worlds/havoc_sim.sdf: new minimal world based on empty.sdf, but with
  the gz-sim-sensors-system and gz-sim-imu-system plugins loaded. The
  stock empty.sdf doesn't load these, so URDF sensor blocks are silent
  until we use a world that does. Will get scenery in a follow-up
  (phase 0.5 of the plan).

- launch/spawn.launch.py: load havoc_sim.sdf instead of empty.sdf.

- config/ros_gz_bridge.yaml: add five new entries to bridge the camera
  topics (image, depth_image, points, camera_info) and the IMU from
  Gazebo to ROS. Existing /cmd_vel bridge entry stays.

- CMakeLists.txt: install the new worlds/ directory.

Verified end-to-end inside the docker ros container (xvfb for headless
sensor rendering):
- ros2 topic list shows /camera/{image,depth_image,points,camera_info}
  and /imu after spawn.
- Publish rates: /imu @ 200 Hz, /camera/image @ ~27 Hz, /camera/points
  @ ~13 Hz. Depth ran low (~4 Hz) under xvfb software rendering; will
  hit target on real GPU.
- TF tree includes base_link -> camera_link -> camera_optical_link and
  base_link -> imu_link, with correct offsets.

This unblocks phase 1 (RTAB-Map mapping a world) and gives target
perception (phase 4) something to look at.

File: ros/src/havoc_description/urdf/havoc.urdf.xacro (robot description, xacro)
@@ -95,4 +95,82 @@
   <xacro:wheel         name="rear_left"   x="${-wheelbase/2.0}" y="${ track/2.0}"/>
   <xacro:wheel         name="rear_right"  x="${-wheelbase/2.0}" y="${-track/2.0}"/>
+  <!-- ====================================================================
+       Depth camera. Mounted at the front of the chassis where the real
+       RealSense D435i will live, tilted ~10 deg down. Two links:
+       camera_link is the physical mount (robot frame, Z-up); the optical
+       frame (Z-forward, Y-down, X-right) is what perception code expects
+       and is what the sensor's published frame_id refers to.
+       ==================================================================== -->
+  <xacro:property name="camera_x"    value="${body_length/2.0 - 0.02}"/>
+  <xacro:property name="camera_z"    value="${wheel_radius + body_height + 0.015}"/>
+  <xacro:property name="camera_tilt" value="0.175"/>  <!-- ~10 deg down -->
+  <link name="camera_link">
+    <inertial>
+      <mass value="0.05"/>
+      <inertia ixx="1e-5" ixy="0" ixz="0" iyy="1e-5" iyz="0" izz="1e-5"/>
+    </inertial>
+    <visual>
+      <geometry><box size="0.025 0.09 0.025"/></geometry>
+      <material name="dark_grey"><color rgba="0.15 0.15 0.15 1"/></material>
+    </visual>
+  </link>
+  <joint name="camera_joint" type="fixed">
+    <parent link="base_link"/>
+    <child  link="camera_link"/>
+    <origin xyz="${camera_x} 0 ${camera_z}" rpy="0 ${camera_tilt} 0"/>
+  </joint>
+  <link name="camera_optical_link"/>
+  <joint name="camera_optical_joint" type="fixed">
+    <parent link="camera_link"/>
+    <child  link="camera_optical_link"/>
+    <origin xyz="0 0 0" rpy="${-pi/2} 0 ${-pi/2}"/>
+  </joint>
+  <gazebo reference="camera_link">
+    <sensor name="rgbd_camera" type="rgbd_camera">
+      <camera>
+        <horizontal_fov>1.21</horizontal_fov>  <!-- ~69 deg, D435i RGB FOV -->
+        <image>
+          <width>640</width>
+          <height>480</height>
+          <format>R8G8B8</format>
+        </image>
+        <clip>
+          <near>0.1</near>
+          <far>10.0</far>
+        </clip>
+        <optical_frame_id>camera_optical_link</optical_frame_id>
+      </camera>
+      <always_on>1</always_on>
+      <update_rate>30</update_rate>
+      <visualize>true</visualize>
+      <topic>camera</topic>
+      <gz_frame_id>camera_optical_link</gz_frame_id>
+    </sensor>
+  </gazebo>
+  <!-- ====================================================================
+       IMU at chassis center. On real hardware this is the MCU-side IMU
+       on the SAM E70's PCB; here it's just a Gazebo IMU sensor publishing
+       acceleration + angular velocity at 200 Hz for SLAM to consume.
+       ==================================================================== -->
+  <link name="imu_link">
+    <inertial>
+      <mass value="0.01"/>
+      <inertia ixx="1e-6" ixy="0" ixz="0" iyy="1e-6" iyz="0" izz="1e-6"/>
+    </inertial>
+  </link>
+  <joint name="imu_joint" type="fixed">
+    <parent link="base_link"/>
+    <child  link="imu_link"/>
+    <origin xyz="0 0 ${wheel_radius + body_height/2.0}"/>
+  </joint>
+  <gazebo reference="imu_link">
+    <sensor name="imu_sensor" type="imu">
+      <always_on>1</always_on>
+      <update_rate>200</update_rate>
+      <visualize>true</visualize>
+      <topic>imu</topic>
+      <gz_frame_id>imu_link</gz_frame_id>
+    </sensor>
+  </gazebo>
   <!-- Gazebo ackermann_steering plugin: drives rear wheels, steers front wheels,
        listens on the gz topic 'cmd_vel' for Twist messages. -->

Commit message: Phase 1.1: SLAM-ready TF tree (odom + base_footprint + joint states)
Sets up the TF chain RTAB-Map needs:
    map -> odom -> base_footprint -> base_link -> camera/imu/wheels

The map->odom edge is reserved for SLAM in 1.2. This PR delivers the
two missing pieces below it.

URDF changes:
- New `base_footprint` link as the URDF root, fixed-joint parent of
  base_link with zero offset. base_footprint sits on the ground plane
  and is the canonical frame for planar odometry.
- Ackermann plugin gets odom emission knobs: <odom_topic>odom</>,
  <tf_topic>tf</>, <frame_id>odom</>, <child_frame_id>base_footprint</>,
  <odom_publish_frequency>50</>.
- New gz-sim-joint-state-publisher-system block so wheel + steer joint
  angles flow as /joint_states. RViz uses these to animate the wheels;
  not required by SLAM but useful for sanity.

Bridge yaml: three new entries
- /odom (nav_msgs/Odometry <-> gz.msgs.Odometry)
- /tf (tf2_msgs/TFMessage <-> gz.msgs.Pose_V) for the dynamic edge
- /joint_states (sensor_msgs/JointState <-> gz.msgs.Model)

Verified end-to-end inside the docker ros container with xvfb:
- /odom publishing at ~46 Hz with frame_id=odom, child=base_footprint.
- /tf carrying the dynamic odom->base_footprint edge at ~33 Hz.
- view_frames shows the full tree connected from odom down through
  camera_optical_link and all 4 wheels.

File: ros/src/havoc_description/urdf/havoc.urdf.xacro (robot description, xacro)
@@ -79,4 +79,15 @@
     </joint>
   </xacro:macro>
+  <!-- base_footprint: a ground-projected frame at z=0 directly below
+       base_link. SLAM and Nav2 want odometry expressed in a planar
+       footprint frame, not the floating chassis. The ackermann plugin
+       publishes odom -> base_footprint and the TF tree then chains up
+       through this static joint to base_link. -->
+  <link name="base_footprint"/>
+  <joint name="base_footprint_joint" type="fixed">
+    <parent link="base_footprint"/>
+    <child  link="base_link"/>
+    <origin xyz="0 0 0"/>
+  </joint>
   <link name="base_link">
     <visual>
@@ -173,6 +184,8 @@
     </sensor>
   </gazebo>
-  <!-- Gazebo ackermann_steering plugin: drives rear wheels, steers front wheels,
-       listens on the gz topic 'cmd_vel' for Twist messages. -->
+  <!-- Gazebo ackermann_steering plugin: drives rear wheels, steers front
+       wheels, listens on the gz topic 'cmd_vel' for Twist messages,
+       publishes odometry (nav_msgs/Odometry-equivalent) and the
+       odom -> base_footprint transform. -->
   <gazebo>
     <plugin filename="gz-sim-ackermann-steering-system"
@@ -188,5 +201,22 @@
       <wheel_radius>${wheel_radius}</wheel_radius>
       <topic>cmd_vel</topic>
+      <!-- Odometry output. SLAM needs odom in a planar footprint frame. -->
+      <odom_topic>odom</odom_topic>
+      <tf_topic>tf</tf_topic>
+      <frame_id>odom</frame_id>
+      <child_frame_id>base_footprint</child_frame_id>
+      <odom_publish_frequency>50</odom_publish_frequency>
     </plugin>
   </gazebo>
+  <!-- Joint state publisher: publishes wheel + steer joint angles so
+       robot_state_publisher can compute live transforms for the wheels
+       and steered links. Without this, the wheels never visibly turn in
+       RViz - they all snap to their zero pose. Doesn't affect SLAM
+       (only odom -> base_footprint matters), but useful for sanity. -->
+  <gazebo>
+    <plugin filename="gz-sim-joint-state-publisher-system"
+            name="gz::sim::systems::JointStatePublisher">
+      <topic>joint_states</topic>
+    </plugin>
+  </gazebo>
 </robot>
